File: 101_BatteryMonitoringUnit_BMU/V_2/KiCAD/BatteryMonitoringUnit_BMU.kicad_pcb (KiCad board)
At the start: 2 copper layers, 106 x 130.8 mm, 155 parts, among them J101 3PinHeader, J102 3PinHeader, J103 2PinHeader, J104 2PinHeader, J105 2PinHeader, J106 2PinHeader, J107 2PinHeader, J108 2PinHeader, J109 2PinHeader, J110 3PinHeader, J1101 3PinHeader, J1102 3PinHeader, J1103 3PinHeader, J1104 3PinHeader, J111 TerminalBlock, J112 Screw_Terminal_01x08, J1301 3PinHeader, J1302 3PinHeader, J1303 3PinHeader, J1304 3PinHeader, J201 2PinHeader, J301 2PinHeader, Q1001 PZT2222A, Q101 DXT5551P5-13, Q401 PZT2222A, Q501 PZT2222A, Q601 PZT2222A, Q701 PZT2222A, Q801 PZT2222A, Q901 PZT2222A, T1201 HM2112ZNL, U101 LTC6810-1_mod, U1101 ADG728, U1102 LTC6255, U1301 24LC256

Commit message: erste platienen bestellt
Parts:
- removed G***: LOGO, myLib:OpenSouceHardwareLOGO
- removed G***: LOGO, myLib:HTWG_LOGO
- added D101: LED_Status, LED_THT:LED_D3.0mm, F.Cu at (52.1, 80.4)
- added L101: LogoHTWG, myLogo:HTWG_LOGO, F.Cu at (118.6, 32.4)
- added L102: LogoOSH, myLogo:OpenSouceHardwareLOGO, F.Cu at (55.4, 59.1)
- added R111: Rv_LED, Resistor_SMD:R_0805_2012Metric_Pad1.20x1.40mm_HandSolder, F.Cu at (60.2, 81.4)
- moved J201 5.99 mm to (109.0, 108.8), turned to 0 degrees
- moved R604 1.34 mm to (70.1, 108.6), turned to 180 degrees
- moved R804 1.34 mm to (93.0, 108.6), turned to 180 degrees
- moved R404 1.34 mm to (47.2, 108.6), turned to 180 degrees
- moved R504 1.34 mm to (58.7, 108.6), turned to 180 degrees
- moved R704 1.34 mm to (81.5, 108.6), turned to 180 degrees
- moved R904 1.34 mm to (104.4, 108.6), turned to 180 degrees
- moved JA101 0.25 mm to (84.3, 32.6)
- moved JB101 0.25 mm to (64.5, 32.6)
Connections:
- JB101 pad SH: Net-(JB101-PadSH) -> Net-(JA101-PadSH)
- R1001 pad 2: -BATT_Fused -> /BalanceFuses/+FusedCell_0
- R109 pad 2: Net-(JB101-PadSH) -> Net-(JA101-PadSH)
- R401 pad 2: /BalanceFuses/+FusedCell_5 -> /BalanceFuses/+FusedCell_6
- R501 pad 2: /BalanceFuses/+FusedCell_4 -> /BalanceFuses/+FusedCell_5
- R601 pad 2: /BalanceFuses/+FusedCell_3 -> /BalanceFuses/+FusedCell_4
- R701 pad 2: /BalanceFuses/+FusedCell_2 -> /BalanceFuses/+FusedCell_3
- R801 pad 2: /BalanceFuses/+FusedCell_1 -> /BalanceFuses/+FusedCell_2
- R901 pad 2: /BalanceFuses/+FusedCell_0 -> /BalanceFuses/+FusedCell_1
Routing:
- net Net-(JA101-PadSH): track 39.3 -> 81.1 mm
- net Net-(JB101-PadSH): track 37.7 -> 0.00 mm
- net /BalanceFuses/+FusedCell_6: track 22.8 -> 40.5 mm
- net /BalanceFuses/+FusedCell_2: track 48.3 -> 55.6 mm, vias 2 -> 4
- net /BalanceFuses/+FusedCell_1: track 48.3 -> 55.6 mm, vias 2 -> 4
- net /BalanceFuses/+FusedCell_5: track 48.3 -> 55.6 mm, vias 2 -> 4
- net /BalanceFuses/+FusedCell_4: track 48.3 -> 55.6 mm, vias 2 -> 4
- net /BalanceFuses/+FusedCell_3: track 48.6 -> 55.6 mm, vias 2 -> 4
- net /BalanceFuses/+FusedCell_0: track 51.1 -> 57.0 mm, vias 2 -> 4
- net -BATT_Fused: track 88.0 -> 93.7 mm
- net Net-(D101-Pad2): track 0.00 -> 5.59 mm
- net /S_1: track 40.2 -> 36.7 mm
- net V_Reg: track 189.0 -> 191.8 mm
- net /S_5: track 32.4 -> 31.4 mm
- net /S_4: track 21.6 -> 20.6 mm
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