File: 101_BatteryMonitoringUnit_BMU/V_2/KiCAD/BatteryMonitoringUnit_BMU.sch (KiCad schematic (older format))
At the start: 43 parts, among them J101 3PinHeader, J102 3PinHeader, J103 2PinHeader, J104 2PinHeader, J105 2PinHeader, J106 2PinHeader, J107 2PinHeader, J108 2PinHeader, J109 2PinHeader, J110 3PinHeader, J111 TerminalBlock, J112 Screw_Terminal_01x08, Q101 DXT5551P5-13, U101 LTC6810-1_mod

Commit message: erste platienen bestellt
Parts:
- added D101: LED_Status, LED_THT:LED_D3.0mm, symbol Device:LED_Small
- added L101: LogoHTWG, myLogo:HTWG_LOGO, symbol myLogo:Logo
- added L102: LogoOSH, myLogo:OpenSouceHardwareLOGO, symbol myLogo:Logo
- added R111: Rv_LED, Resistor_SMD:R_0805_2012Metric_Pad1.20x1.40mm_HandSolder, symbol Device:R_Small
Connections:
- net +5V: now also R111.1
- net -BATT_Fused: now also D101.1 (K)
- net at JB101.SH, R109.2: now also JA101.SH, R110.2
- new net: D101.2 (A), R111.2
Other:
- note removed: "https://componentsearchengine.com/"
Changed lines of the file:
@@
 Wire Wire Line
 	10250 3350 10250 3400
-Text Notes 9550 7350 0    50   ~ 0
-https://componentsearchengine.com/
 Wire Wire Line
 	1000 4050 1000 4250
@@
 $EndComp
 Wire Wire Line
-	10550 2100 10250 2100
-Wire Wire Line
 	10250 3350 10550 3350
 $Comp
@@
 Wire Wire Line
 	7300 3700 7550 3700
+Wire Wire Line
+	10250 2100 10550 2100
+Wire Wire Line
+	10250 2150 10600 2150
+Wire Wire Line
+	10600 2150 10600 3300
+Wire Wire Line
+	10600 3300 10250 3300
+Wire Wire Line
+	10250 3300 10250 3350
+Connection ~ 10250 2150
+Connection ~ 10250 3350
+Text GLabel 1400 1850 0    50   Input ~ 0
+V_Reg
+$Comp
+L Device:LED_Small D?
+U 1 1 5FA17A47
+P 1450 2250
+AR Path="/5F9A2BC6/5FD0CC74/5FA17A47" Ref="D?"  Part="1"
+AR Path="/5F9A2BC6/5FD73853/5FA17A47" Ref="D?"  Part="1"
+AR Path="/5F9A2BC6/5FD7394A/5FA17A47" Ref="D?"  Part="1"
+AR Path="/5F9A2BC6/5FD74270/5FA17A47" Ref="D?"  Part="1"
+AR Path="/5F9A2BC6/5FD74408/5FA17A47" Ref="D?"  Part="1"
+AR Path="/5F9A2BC6/5FD74551/5FA17A47" Ref="D?"  Part="1"
+AR Path="/5F9A2BC6/5FD749CA/5FA17A47" Ref="D?"  Part="1"
+AR Path="/5F9A2BC6/5FD7C7E7/5FA17A47" Ref="D?"  Part="1"
+AR Path="/5F9A2BC6/5F981FE3/5FA17A47" Ref="D?"  Part="1"
+AR Path="/5F9A2BC6/5F9823BC/5FA17A47" Ref="D?"  Part="1"
+AR Path="/5F9A2BC6/5F982EA0/5FA17A47" Ref="D?"  Part="1"
+AR Path="/5F9A2BC6/5F9831DE/5FA17A47" Ref="D?"  Part="1"
+AR Path="/5F9A2BC6/5F983535/5FA17A47" Ref="D?"  Part="1"
+AR Path="/5F9A2BC6/5F983909/5FA17A47" Ref="D?"  Part="1"
+AR Path="/5F9A2BC6/5F983C60/5FA17A47" Ref="D?"  Part="1"
+AR Path="/5F9A2BC6/5F983FE9/5FA17A47" Ref="D?"  Part="1"
+AR Path="/5F9A2BC6/5FE0CA77/5FA17A47" Ref="D?"  Part="1"
+AR Path="/5F9A2BC6/5FE0D3F9/5FA17A47" Ref="D?"  Part="1"
+AR Path="/5F9A2BC6/5FE0DD76/5FA17A47" Ref="D?"  Part="1"
+AR Path="/5F9A2BC6/5FE0E6D5/5FA17A47" Ref="D?"  Part="1"
+AR Path="/5F9A2BC6/5FE0F048/5FA17A47" Ref="D?"  Part="1"
+AR Path="/5F9A2BC6/5FE0FA0B/5FA17A47" Ref="D?"  Part="1"
+AR Path="/5FA17A47" Ref="D101"  Part="1"
+F 0 "D101" V 1496 2180 50  0000 R CNN
+F 1 "LED_Status" V 1405 2180 50  0000 R CNN
+F 2 "LED_THT:LED_D3.0mm" V 1450 2250 50  0001 C CNN
+F 3 "~" V 1450 2250 50  0001 C CNN
+	1    1450 2250
+	0    -1   -1   0
+$EndComp
+$Comp
+L Device:R_Small R?
+U 1 1 5FA17A4D
+P 1450 2050
+AR Path="/5F9A2BC6/5FD0CC74/5FA17A4D" Ref="R?"  Part="1"
+AR Path="/5F9A2BC6/5FD73853/5FA17A4D" Ref="R?"  Part="1"
+AR Path="/5F9A2BC6/5FD7394A/5FA17A4D" Ref="R?"  Part="1"
+AR Path="/5F9A2BC6/5FD74270/5FA17A4D" Ref="R?"  Part="1"
+AR Path="/5F9A2BC6/5FD74408/5FA17A4D" Ref="R?"  Part="1"
+AR Path="/5F9A2BC6/5FD74551/5FA17A4D" Ref="R?"  Part="1"
+AR Path="/5F9A2BC6/5FD749CA/5FA17A4D" Ref="R?"  Part="1"
+AR Path="/5F9A2BC6/5FD7C7E7/5FA17A4D" Ref="R?"  Part="1"
+AR Path="/5F9A2BC6/5F981FE3/5FA17A4D" Ref="R?"  Part="1"
+AR Path="/5F9A2BC6/5F9823BC/5FA17A4D" Ref="R?"  Part="1"
+AR Path="/5F9A2BC6/5F982EA0/5FA17A4D" Ref="R?"  Part="1"
+AR Path="/5F9A2BC6/5F9831DE/5FA17A4D" Ref="R?"  Part="1"
+AR Path="/5F9A2BC6/5F983535/5FA17A4D" Ref="R?"  Part="1"
+AR Path="/5F9A2BC6/5F983909/5FA17A4D" Ref="R?"  Part="1"
+AR Path="/5F9A2BC6/5F983C60/5FA17A4D" Ref="R?"  Part="1"
+AR Path="/5F9A2BC6/5F983FE9/5FA17A4D" Ref="R?"  Part="1"
+AR Path="/5F9A2BC6/5FE0CA77/5FA17A4D" Ref="R?"  Part="1"
+AR Path="/5F9A2BC6/5FE0D3F9/5FA17A4D" Ref="R?"  Part="1"
+AR Path="/5F9A2BC6/5FE0DD76/5FA17A4D" Ref="R?"  Part="1"
+AR Path="/5F9A2BC6/5FE0E6D5/5FA17A4D" Ref="R?"  Part="1"
+AR Path="/5F9A2BC6/5FE0F048/5FA17A4D" Ref="R?"  Part="1"
+AR Path="/5F9A2BC6/5FE0FA0B/5FA17A4D" Ref="R?"  Part="1"
+AR Path="/5FA17A4D" Ref="R111"  Part="1"
+F 0 "R111" H 1509 2096 50  0000 L CNN
+F 1 "Rv_LED" H 1509 2005 50  0000 L CNN
+F 2 "Resistor_SMD:R_0805_2012Metric_Pad1.20x1.40mm_HandSolder" H 1450 2050 50  0001 C CNN
+F 3 "~" H 1450 2050 50  0001 C CNN
+	1    1450 2050
+	1    0    0    -1
+$EndComp
+$Comp
+L myPower:-BATT_Fused #PWR0129
+U 1 1 5FA26F73
+P 1450 2400
+F 0 "#PWR0129" H 1450 2250 50  0001 C CNN
+F 1 "-BATT_Fused" H 1465 2573 50  0000 C CNN
+F 2 "" H 1450 2400 50  0001 C CNN
+F 3 "" H 1450 2400 50  0001 C CNN
+	1    1450 2400
+	-1   0    0    1
+$EndComp
+Wire Wire Line
+	1400 1850 1450 1850
+Wire Wire Line
+	1450 1850 1450 1950
+Wire Wire Line
+	1450 2350 1450 2400
+$Comp
+L myLogo:Logo L101
+U 1 1 5FA31AFD
+P 4250 7000
+F 0 "L101" H 4275 7046 50  0000 L CNN
+F 1 "LogoHTWG" H 4275 6955 50  0000 L CNN
+F 2 "myLogo:HTWG_LOGO" H 4250 7000 50  0001 C CNN
+F 3 "" H 4250 7000 50  0001 C CNN
+	1    4250 7000
+	1    0    0    -1
+$EndComp
+$Comp
+L myLogo:Logo L102
+U 1 1 5FA6162B
+P 4750 7000
+F 0 "L102" H 4775 7046 50  0000 L CNN
+F 1 "LogoOSH" H 4775 6955 50  0000 L CNN
+F 2 "myLogo:OpenSouceHardwareLOGO" H 4750 7000 50  0001 C CNN
+F 3 "" H 4750 7000 50  0001 C CNN
+	1    4750 7000
+	1    0    0    -1
+$EndComp
 Wire Bus Line
 	9600 6050 9600 6400
