File: 101_BatteryMonitoringUnit_BMU/V_2/KiCAD/SingleCellCircuit.sch (KiCad schematic (older format))
At the start: 8 parts, among them Q401 PZT2222A

Commit message: erste platienen bestellt
Connections:
- net Cell+: now also R401.2
- net Cell-: no longer R401.2
Other:
- note added: "use PFET if 7 Cell"
- moved on the sheet: C1001, R1001
Changed lines of the file:
@@
 $Descr A4 11693 8268
 encoding utf-8
-Sheet 4 13
+Sheet 10 13
 Title "Battery Monitoring Unit"
 Date "2020-10-28"
@@
 Comment4 ""
 $EndDescr
-Connection ~ 1750 3200
-Wire Wire Line
-	1750 3200 1250 3200
-Wire Wire Line
-	1750 3200 1750 3250
-Wire Wire Line
-	1800 3200 1750 3200
-Wire Wire Line
-	1750 3500 1750 3450
+Connection ~ 1650 3150
+Wire Wire Line
+	1650 3150 2150 3150
+Wire Wire Line
+	1650 3150 1650 3200
+Wire Wire Line
+	1600 3150 1650 3150
+Wire Wire Line
+	1650 3450 1650 3400
 $Comp
 L Device:C_Small C401
 U 1 1 5FD1663D
-P 1750 3350
+P 1650 3300
 AR Path="/5F9A2BC6/5FD0CC74/5FD1663D" Ref="C401"  Part="1"
 AR Path="/5F9A2BC6/5FD73853/5FD1663D" Ref="C?"  Part="1"
@@
 AR Path="/5F9A2BC6/5FE0F048/5FD1663D" Ref="C901"  Part="1"
 AR Path="/5F9A2BC6/5FE0FA0B/5FD1663D" Ref="C1001"  Part="1"
-F 0 "C401" H 1842 3396 50  0000 L CNN
-F 1 "10nF/30V" H 1842 3305 50  0000 L CNN
-F 2 "Capacitor_SMD:C_0805_2012Metric_Pad1.18x1.45mm_HandSolder" H 1750 3350 50  0001 C CNN
-F 3 "~" H 1750 3350 50  0001 C CNN
-	1    1750 3350
-	-1   0    0    -1
-$EndComp
-Text HLabel 1250 3200 0    50   BiDi ~ 0
+F 0 "C1001" H 1742 3346 50  0000 L CNN
+F 1 "10nF/30V" H 1742 3255 50  0000 L CNN
+F 2 "Capacitor_SMD:C_0805_2012Metric_Pad1.18x1.45mm_HandSolder" H 1650 3300 50  0001 C CNN
+F 3 "~" H 1650 3300 50  0001 C CNN
+	1    1650 3300
+	1    0    0    -1
+$EndComp
+Text HLabel 2150 3150 2    50   BiDi ~ 0
 C_(n)
 $Comp
 L Device:R_Small R401
 U 1 1 5FD15F7A
-P 1900 3200
+P 1500 3150
 AR Path="/5F9A2BC6/5FD0CC74/5FD15F7A" Ref="R401"  Part="1"
 AR Path="/5F9A2BC6/5FD73853/5FD15F7A" Ref="R?"  Part="1"
@@
 AR Path="/5F9A2BC6/5FE0F048/5FD15F7A" Ref="R901"  Part="1"
 AR Path="/5F9A2BC6/5FE0FA0B/5FD15F7A" Ref="R1001"  Part="1"
-F 0 "R401" V 1704 3200 50  0000 C CNN
-F 1 "100" V 1795 3200 50  0000 C CNN
-F 2 "Resistor_SMD:R_0805_2012Metric_Pad1.20x1.40mm_HandSolder" H 1900 3200 50  0001 C CNN
-F 3 "~" H 1900 3200 50  0001 C CNN
-	1    1900 3200
-	0    -1   1    0
-$EndComp
-Wire Wire Line
-	2150 3200 2000 3200
+F 0 "R1001" V 1304 3150 50  0000 C CNN
+F 1 "100" V 1395 3150 50  0000 C CNN
+F 2 "Resistor_SMD:R_0805_2012Metric_Pad1.20x1.40mm_HandSolder" H 1500 3150 50  0001 C CNN
+F 3 "~" H 1500 3150 50  0001 C CNN
+	1    1500 3150
+	0    1    1    0
+$EndComp
+Wire Wire Line
+	1250 3150 1400 3150
 Wire Notes Line
 	3250 800  3250 2700
@@
 Text Notes 1750 2950 2    50   ~ 0
 Voltage Measurement\n
-Text HLabel 2150 3200 2    50   Output ~ 0
-Cell-
 Text Notes 3500 1350 0    50   ~ 0
 @50 Ohm\n5V -> 100mA Balancing Current\n4V ->  80mA Balancing Current\n3V ->  60mA Balancing Current\n2V ->  40mA Balancing Current
@@
 AR Path="/5F9A2BC6/5FE0F048/605B7E40" Ref="D901"  Part="1"
 AR Path="/5F9A2BC6/5FE0FA0B/605B7E40" Ref="D1001"  Part="1"
-F 0 "D401" V 2596 1430 50  0000 R CNN
+F 0 "D1001" V 2596 1430 50  0000 R CNN
 F 1 "LED_Dis" V 2505 1430 50  0000 R CNN
 F 2 "LED_THT:LED_D3.0mm" V 2550 1500 50  0001 C CNN
@@
 AR Path="/5F9A2BC6/5FE0F048/605B7E46" Ref="R905"  Part="1"
 AR Path="/5F9A2BC6/5FE0FA0B/605B7E46" Ref="R1005"  Part="1"
-F 0 "R405" H 2609 1346 50  0000 L CNN
+F 0 "R1005" H 2609 1346 50  0000 L CNN
 F 1 "Rv_LED" H 2609 1255 50  0000 L CNN
 F 2 "Resistor_SMD:R_0805_2012Metric_Pad1.20x1.40mm_HandSolder" H 2550 1300 50  0001 C CNN
@@
 AR Path="/5F9A2BC6/5FE0F048/605BBB1B" Ref="R903"  Part="1"
 AR Path="/5F9A2BC6/5FE0FA0B/605BBB1B" Ref="R1003"  Part="1"
-F 0 "R403" H 1800 1450 50  0000 L CNN
+F 0 "R1003" H 1800 1450 50  0000 L CNN
 F 1 "100" H 1800 1350 50  0000 L CNN
 F 2 "Resistor_SMD:R_2512_6332Metric_Pad1.40x3.35mm_HandSolder" V 2030 1400 50  0001 C CNN
@@
 AR Path="/5F9A2BC6/5FE0F048/605BBB21" Ref="R902"  Part="1"
 AR Path="/5F9A2BC6/5FE0FA0B/605BBB21" Ref="R1002"  Part="1"
-F 0 "R402" H 1700 1450 50  0000 L CNN
+F 0 "R1002" H 1700 1450 50  0000 L CNN
 F 1 "100" H 1700 1350 50  0000 L CNN
 F 2 "Resistor_SMD:R_2512_6332Metric_Pad1.40x3.35mm_HandSolder" V 1930 1400 50  0001 C CNN
@@
 AR Path="/5F9A2BC6/5FE0F048/605BE3F6" Ref="R904"  Part="1"
 AR Path="/5F9A2BC6/5FE0FA0B/605BE3F6" Ref="R1004"  Part="1"
-F 0 "R404" V 2054 2200 50  0000 C CNN
+F 0 "R1004" V 2054 2200 50  0000 C CNN
 F 1 "1k" V 2145 2200 50  0000 C CNN
 F 2 "Resistor_SMD:R_0805_2012Metric_Pad1.20x1.40mm_HandSolder" H 2250 2200 50  0001 C CNN
@@
 	2600 1900 2400 1900
 Connection ~ 2400 1900
-Text HLabel 1600 1150 0    50   Input ~ 0
+Text HLabel 1250 3150 0    50   Input ~ 0
 Cell+
 Connection ~ 2050 1150
@@
 AR Path="/5F9A2BC6/5FE0F048/5FA411D8" Ref="Q901"  Part="1"
 AR Path="/5F9A2BC6/5FE0FA0B/5FA411D8" Ref="Q1001"  Part="1"
-F 0 "Q401" H 2341 1946 50  0000 L CNN
+F 0 "Q1001" H 2341 1946 50  0000 L CNN
 F 1 "PZT2222A" H 2341 1855 50  0000 L CNN
 F 2 "Package_TO_SOT_SMD:SOT-223-3_TabPin2" H 2350 1825 50  0001 L CIN
@@
 L myPower:-BATT_Fused #PWR?
 U 1 1 601ABE72
-P 1750 3500
+P 1650 3450
 AR Path="/601ABE72" Ref="#PWR?"  Part="1"
 AR Path="/5F9A2BC6/5FD0CC74/601ABE72" Ref="#PWR0401"  Part="1"
@@
 AR Path="/5F9A2BC6/5FE0F048/601ABE72" Ref="#PWR0901"  Part="1"
 AR Path="/5F9A2BC6/5FE0FA0B/601ABE72" Ref="#PWR01001"  Part="1"
-F 0 "#PWR0401" H 1750 3350 50  0001 C CNN
-F 1 "-BATT_Fused" H 1765 3673 50  0000 C CNN
-F 2 "" H 1750 3500 50  0001 C CNN
-F 3 "" H 1750 3500 50  0001 C CNN
-	1    1750 3500
-	-1   0    0    1
-$EndComp
+F 0 "#PWR01001" H 1650 3300 50  0001 C CNN
+F 1 "-BATT_Fused" H 1665 3623 50  0000 C CNN
+F 2 "" H 1650 3450 50  0001 C CNN
+F 3 "" H 1650 3450 50  0001 C CNN
+	1    1650 3450
+	1    0    0    1
+$EndComp
+Text HLabel 1600 1150 0    50   Input ~ 0
+Cell+
+Text Notes 3350 2050 0    50   ~ 0
+use PFET if 7 Cell
 $EndSCHEMATC
