File: 111_7CellBatterySimulator_7CBS/KiCAD/7CellBatterySimulator_7CBS.sch (KiCad schematic (older format))
At the start: 11 parts, among them J101 Screw_Terminal_01x02, J102 Screw_Terminal_01x08

Commit message: erste platienen bestellt
Parts:
- added L101: LogoHTWG, myLogo:HTWG_LOGO, symbol myLogo:Logo
- added L102: LogoOSH, myLogo:OpenSouceHardwareLOGO, symbol myLogo:Logo
Changed lines of the file:
@@
 Wire Wire Line
 	6100 1650 6100 1450
+$Comp
+L myLogo:Logo L102
+U 1 1 5FA0457A
+P 2150 4850
+F 0 "L102" H 2175 4896 50  0000 L CNN
+F 1 "LogoOSH" H 2175 4805 50  0000 L CNN
+F 2 "myLogo:OpenSouceHardwareLOGO" H 2150 4850 50  0001 C CNN
+F 3 "" H 2150 4850 50  0001 C CNN
+	1    2150 4850
+	1    0    0    -1
+$EndComp
+$Comp
+L myLogo:Logo L101
+U 1 1 5FA04AA8
+P 2150 4450
+F 0 "L101" H 2175 4496 50  0000 L CNN
+F 1 "LogoHTWG" H 2175 4405 50  0000 L CNN
+F 2 "myLogo:HTWG_LOGO" H 2150 4450 50  0001 C CNN
+F 3 "" H 2150 4450 50  0001 C CNN
+	1    2150 4450
+	1    0    0    -1
+$EndComp
 $EndSCHEMATC
