File: 111_7CellBatterySimulator_7CBS/KiCAD/7CellBatterySimulator_7CBS.kicad_pcb (KiCad board)
At the start: 2 copper layers, 123.8 x 140.3 mm, 85 parts, among them J101 Screw_Terminal_01x02, J102 Screw_Terminal_01x08, U201 LM317_SOT-223, U301 LM317_SOT-223, U401 LM317_SOT-223, U501 LM317_SOT-223, U601 LM317_SOT-223, U701 LM317_SOT-223, U801 LM317_SOT-223

Commit message: erste platienen bestellt
Parts:
- removed G***: LOGO, myLib:OpenSouceHardwareLOGO_F-CU
- removed G***: LOGO, myLib:OpenSouceHardwareLOGO
- removed G***: LOGO, myLib:HTWG_LOGO_F-CU
- removed G***: LOGO, myLib:HTWG_LOGO
- added L101: LogoHTWG, myLogo:HTWG_LOGO, F.Cu at (156.7, 40.9)
- added L102: LogoOSH, myLogo:OpenSouceHardwareLOGO, F.Cu at (156.2, 145.5)
- D101: value 40V 2A -> 60V; footprint Diode_SMD:D_1206_3216Metric_Pad1.42x1.75mm_HandSolder -> Diode_SMD:D_3220_8050Metric_Pad2.65x5.15mm_HandSolder
- J101: footprint TerminalBlock_Phoenix:TerminalBlock_Phoenix_MKDS-3-2-5.08_1x02_P5.08mm_Horizontal -> TerminalBlock_Phoenix:TerminalBlock_Phoenix_PT-1,5-2-5.0-H_1x02_P5.00mm_Horizontal
- moved D102 2.36 mm to (67.3, 25.9)
- moved R101 1.78 mm to (64.4, 37.1)
Routing:
- net Net-(D102-Pad2): track 4.96 -> 9.20 mm
- net +5V: track 199.9 -> 203.9 mm
- net Net-(D101-Pad2): track 5.08 -> 5.82 mm

Commit message: some small chages in 7CBS
Other:
- net class Default: via_dia 0.8 -> 0.9
- rule via_min_size: 0.4 -> 0.6
