File: 120_isoSPI_Interface/KiCAD/isoSPI_Interface.kicad_pcb (KiCad board)
At the start: 2 copper layers, 50.8 x 88.9 mm, 47 parts, among them IC201 LTC6820IMS#PBF, IC401 LTC6820IMS#PBF, J101 Conn_01x02_Male, J102 RJ45_Shielded_1, J103 Conn_01x07_Male, J104 RJ45_Shielded_2, J201 3PinHeader, J202 3PinHeader, J203 3PinHeader, J204 3PinHeader, J205 3PinHeader, J401 3PinHeader, J402 3PinHeader, J403 3PinHeader, J404 3PinHeader, J405 3PinHeader, T301 HM2112ZNL

Commit message: erste platienen bestellt
Parts:
- added L101: LogoHTWG, myLogo:HTWG_LOGO, F.Cu at (104.1, 131.8)
- added L102: LogoOSH, myLogo:OpenSouceHardwareLOGO, F.Cu at (133.3, 131.1)
- moved H103 1.65 mm to (138.2, 109.2)
- moved H101 1.27 mm to (96.5, 109.1)
Connections:
- J104 pad SH: Net-(J104-PadSH) -> Net-(J102-PadSH)
- R103 pad 2: Net-(J104-PadSH) -> Net-(J102-PadSH)
Routing:
- net Net-(J102-PadSH): track 68.4 -> 166.4 mm
- net Net-(J104-PadSH): track 68.7 -> 0.00 mm
Other:
- board text added: "isoSPI-SPI Interface"
- board text removed: "isoSPI <-> SPI Interface"
