File: 103_BatteryJunctionBox_BJB/KiCAD/V0_1/IsoPowerSupply.sch (KiCad schematic (older format))
At the start: 12 parts

Commit message: Mon. Done a Lot of recouvery
Parts:
- L301: renamed from L?; footprint (none) -> Inductor_THT:L_Radial_D12.0mm_P6.00mm_MuRATA_1900R
- PS301: renamed from PS?; footprint RI0505S -> _Package_SIP:SIP4_SingleOutput
- R301, R302, R303: renamed from R?; footprint Resistor_SMD:R_0815_2038Metric_Pad1.20x4.05mm_HandSolder -> Resistor_SMD:R_0805_2012Metric_Pad1.20x1.40mm_HandSolder
- gave numbers to parts that had none: 7
Changed lines of the file:
@@
 $EndDescr
 $Comp
-L _Power_ICs:LT8630IFE#PBF IC?
+L _Power_ICs:LT8630IFE#PBF IC301
 U 1 1 5FAABA2E
 P 4650 1350
-F 0 "IC?" H 5350 1615 50  0000 C CNN
+F 0 "IC301" H 5350 1615 50  0000 C CNN
 F 1 "LT8630IFE#PBF" H 5350 1524 50  0000 C CNN
 F 2 "_Package_SMDSpecial:LT8630IFEPBF" H 5900 1450 50  0001 L CNN
@@
 P 4250 1500
 AR Path="/5FA7E0E6/5FAAD5E6" Ref="C?"  Part="1"
-AR Path="/5FAAB734/5FAAD5E6" Ref="C?"  Part="1"
-F 0 "C?" H 4158 1454 50  0000 R CNN
+AR Path="/5FAAB734/5FAAD5E6" Ref="C302"  Part="1"
+F 0 "C302" H 4158 1454 50  0000 R CNN
 F 1 "2.2u" H 4158 1545 50  0000 R CNN
 F 2 "Capacitor_SMD:C_0805_2012Metric_Pad1.18x1.45mm_HandSolder" H 4250 1500 50  0001 C CNN
@@
 P 6600 1750
 AR Path="/5FA7E0E6/5FAB0422" Ref="C?"  Part="1"
-AR Path="/5FAAB734/5FAB0422" Ref="C?"  Part="1"
-F 0 "C?" V 6829 1750 50  0000 C CNN
+AR Path="/5FAAB734/5FAB0422" Ref="C303"  Part="1"
+F 0 "C303" V 6829 1750 50  0000 C CNN
 F 1 "2.2u" V 6738 1750 50  0000 C CNN
 F 2 "Capacitor_SMD:C_0805_2012Metric_Pad1.18x1.45mm_HandSolder" H 6600 1750 50  0001 C CNN
@@
 P 6150 1450
 AR Path="/5FA7E0E6/5FAB2C8B" Ref="C?"  Part="1"
-AR Path="/5FAAB734/5FAB2C8B" Ref="C?"  Part="1"
-F 0 "C?" H 6242 1496 50  0000 L CNN
+AR Path="/5FAAB734/5FAB2C8B" Ref="C301"  Part="1"
+F 0 "C301" H 6242 1496 50  0000 L CNN
 F 1 "0.1u" H 6242 1405 50  0000 L CNN
 F 2 "Capacitor_SMD:C_0805_2012Metric_Pad1.18x1.45mm_HandSolder" H 6150 1450 50  0001 C CNN
@@
 $EndComp
 $Comp
-L Device:L L?
+L Device:L L301
 U 1 1 5FAB3F96
 P 6550 1350
-F 0 "L?" V 6740 1350 50  0000 C CNN
+F 0 "L301" V 6740 1350 50  0000 C CNN
 F 1 "22u" V 6649 1350 50  0000 C CNN
-F 2 "" H 6550 1350 50  0001 C CNN
+F 2 "Inductor_THT:L_Radial_D12.0mm_P6.00mm_MuRATA_1900R" H 6550 1350 50  0001 C CNN
 F 3 "~" H 6550 1350 50  0001 C CNN
 	1    6550 1350
@@
 P 6250 2250
 AR Path="/5FA7E0E6/5FAB5144" Ref="C?"  Part="1"
-AR Path="/5FAAB734/5FAB5144" Ref="C?"  Part="1"
-F 0 "C?" H 6158 2204 50  0000 R CNN
+AR Path="/5FAAB734/5FAB5144" Ref="C304"  Part="1"
+F 0 "C304" H 6158 2204 50  0000 R CNN
 F 1 "10p" H 6158 2295 50  0000 R CNN
 F 2 "Capacitor_SMD:C_0805_2012Metric_Pad1.18x1.45mm_HandSolder" H 6250 2250 50  0001 C CNN
@@
 P 6600 2250
 AR Path="/5FA7E0E6/5FAB7244" Ref="R?"  Part="1"
-AR Path="/5FAAB734/5FAB7244" Ref="R?"  Part="1"
-F 0 "R?" H 6659 2296 50  0000 L CNN
+AR Path="/5FAAB734/5FAB7244" Ref="R301"  Part="1"
+F 0 "R301" H 6659 2296 50  0000 L CNN
 F 1 "1Mega" H 6659 2205 50  0000 L CNN
-F 2 "Resistor_SMD:R_0815_2038Metric_Pad1.20x4.05mm_HandSolder" H 6600 2250 50  0001 C CNN
+F 2 "Resistor_SMD:R_0805_2012Metric_Pad1.20x1.40mm_HandSolder" H 6600 2250 50  0001 C CNN
 F 3 "~" H 6600 2250 50  0001 C CNN
 	1    6600 2250
@@
 P 6600 2450
 AR Path="/5FA7E0E6/5FAB7DA7" Ref="R?"  Part="1"
-AR Path="/5FAAB734/5FAB7DA7" Ref="R?"  Part="1"
-F 0 "R?" H 6659 2496 50  0000 L CNN
+AR Path="/5FAAB734/5FAB7DA7" Ref="R303"  Part="1"
+F 0 "R303" H 6659 2496 50  0000 L CNN
 F 1 "71.5k" H 6659 2405 50  0000 L CNN
-F 2 "Resistor_SMD:R_0815_2038Metric_Pad1.20x4.05mm_HandSolder" H 6600 2450 50  0001 C CNN
+F 2 "Resistor_SMD:R_0805_2012Metric_Pad1.20x1.40mm_HandSolder" H 6600 2450 50  0001 C CNN
 F 3 "~" H 6600 2450 50  0001 C CNN
 	1    6600 2450
@@
 P 4500 2400
 AR Path="/5FA7E0E6/5FAB934D" Ref="C?"  Part="1"
-AR Path="/5FAAB734/5FAB934D" Ref="C?"  Part="1"
-F 0 "C?" H 4592 2446 50  0000 L CNN
+AR Path="/5FAAB734/5FAB934D" Ref="C306"  Part="1"
+F 0 "C306" H 4592 2446 50  0000 L CNN
 F 1 "0.1u" H 4592 2355 50  0000 L CNN
 F 2 "Capacitor_SMD:C_0805_2012Metric_Pad1.18x1.45mm_HandSolder" H 4500 2400 50  0001 C CNN
@@
 P 4150 2400
 AR Path="/5FA7E0E6/5FABA3AB" Ref="R?"  Part="1"
-AR Path="/5FAAB734/5FABA3AB" Ref="R?"  Part="1"
-F 0 "R?" H 4209 2446 50  0000 L CNN
+AR Path="/5FAAB734/5FABA3AB" Ref="R302"  Part="1"
+F 0 "R302" H 4209 2446 50  0000 L CNN
 F 1 "8.66k" H 4209 2355 50  0000 L CNN
-F 2 "Resistor_SMD:R_0815_2038Metric_Pad1.20x4.05mm_HandSolder" H 4150 2400 50  0001 C CNN
+F 2 "Resistor_SMD:R_0805_2012Metric_Pad1.20x1.40mm_HandSolder" H 4150 2400 50  0001 C CNN
 F 3 "~" H 4150 2400 50  0001 C CNN
 	1    4150 2400
@@
 P 7250 2250
 AR Path="/5FA7E0E6/5FAC0FDE" Ref="C?"  Part="1"
-AR Path="/5FAAB734/5FAC0FDE" Ref="C?"  Part="1"
-F 0 "C?" H 7158 2204 50  0000 R CNN
+AR Path="/5FAAB734/5FAC0FDE" Ref="C305"  Part="1"
+F 0 "C305" H 7158 2204 50  0000 R CNN
 F 1 "47u" H 7158 2295 50  0000 R CNN
 F 2 "Capacitor_SMD:C_0805_2012Metric_Pad1.18x1.45mm_HandSolder" H 7250 2250 50  0001 C CNN
@@
 NoConn ~ 4650 1750
 $Comp
-L _DC-DC-Wandler:RI-1205S PS?
+L _DC-DC-Wandler:RI-1205S PS301
 U 1 1 5FACE5AF
 P 5200 4500
-F 0 "PS?" V 5683 4072 50  0000 R CNN
+F 0 "PS301" V 5683 4072 50  0000 R CNN
 F 1 "RI-1205S" V 5592 4072 50  0000 R CNN
-F 2 "RI0505S" H 6050 4600 50  0001 L CNN
+F 2 "_Package_SIP:SIP4_SingleOutput" H 6050 4600 50  0001 L CNN
 F 3 "https://www.mouser.de/datasheet/2/468/RI-1711294.pdf" H 6050 4500 50  0001 L CNN
 F 4 "Recom 2W Isolated DC-DC Converter, Vin 10.8  13.2 V dc, Vout 5V dc, I/O isolation 1000V" H 6050 4400 50  0001 L CNN "Description"
