File: 103_BatteryJunctionBox_BJB/KiCAD/V0_1/BatteryJunctionBox_BJB.kicad_pcb (KiCad board)
At the start: 2 copper layers, 33 parts, among them IC101 VOM1271T, IC201 LTC2946, IC301 LT8630IFE#PBF, J101 WuertHA_7461057, J102 WuertHA_7461057, J103 WuertHA_7461057, J104 WuertHA_7461057, J105 RJ45_Shielded, Q101 Q_NMOS_GDS, Q102 Q_NMOS_GDS, Q103 Q_NMOS_GDS, Q104 Q_NMOS_GDS, U101 NSL-32, U102 ISO1541

Commit message: some small chages in 7CBS
Parts:
- moved C306 120.5 mm to (39.5, 40.1), turned to 90 degrees
- moved C302 116.5 mm to (45.3, 40.1), turned to 270 degrees
- moved R302 116.4 mm to (41.5, 40.1), turned to 90 degrees
- moved C303 113.2 mm to (42.7, 53.1), turned to 270 degrees
- moved C301 112.3 mm to (45.6, 52.2), turned to 180 degrees
- moved IC301 110.1 mm to (42.4, 46.7), turned to 180 degrees
- moved C304 109.1 mm to (38.8, 52.3)
- moved J104 106.3 mm to (114.2, 66.5)
- moved C305 105.3 mm to (38.8, 56.6)
- moved U102 105.2 mm to (63.2, 75.2), turned to 90 degrees
- moved R303 104.8 mm to (35.8, 55.8), turned to 270 degrees
- moved J105 101.1 mm to (84.3, 79.8), turned to 180 degrees
- moved R301 99.0 mm to (38.8, 54.5), turned to 180 degrees
- moved R102 96.4 mm to (60.8, 49.3), turned to 180 degrees
- moved R103 90.1 mm to (61.7, 51.8), turned to 180 degrees
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Connections:
- C302 pad 2: SHUNT+ -> +BATT
- IC201 pad 1: SHUNT+ -> +BATT
- IC301 pad 1: SHUNT+ -> +BATT
- IC301 pad 3: SHUNT+ -> +BATT
- J101 pad 1: SHUNT+ -> +BATT
- J101 pad 2: SHUNT+ -> +BATT
- J101 pad 3: SHUNT+ -> +BATT
- J101 pad 4: SHUNT+ -> +BATT
- J101 pad 5: SHUNT+ -> +BATT
- J101 pad 6: SHUNT+ -> +BATT
- Q101 pad 2: SHUNT- -> Net-(Q101-Pad2)
- Q103 pad 2: SHUNT- -> Net-(Q101-Pad2)
- R101 pad 1: SHUNT+ -> +BATT
- R101 pad 4: SHUNT- -> Net-(Q101-Pad2)
- R201 pad 1: SHUNT+ -> +BATT
Routing:
- net ISO_GND: track 0.00 -> 59.7 mm
- net -BATT: track 0.00 -> 41.6 mm, vias 0 -> 2
- net I2C_SDA: track 0.00 -> 35.3 mm
- net +BATT: track 0.00 -> 30.2 mm
- net I2C_SCL: track 0.00 -> 30.2 mm
- net /IsoPowerSupply/12V_OUT: track 0.00 -> 29.0 mm
- net ~ALERT: track 0.00 -> 25.5 mm
- net MOSFET_G: track 51.1 -> 70.6 mm, vias 4 -> 5
- net MOSFET_S: track 51.1 -> 69.3 mm, vias 4 -> 5
- net Net-(IC301-Pad14): track 0.00 -> 15.9 mm
- net MOSFET_SWITCH: track 0.00 -> 13.5 mm
- net SHUNT+: track 23.4 -> 10.1 mm
- net +5V: track 2.37 -> 14.3 mm
- net +3V3: track 0.00 -> 11.4 mm
- net /PowerMonitor/ADIN: track 20.1 -> 10.2 mm
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- added copper zone on F.Cu, net +BATT
- added copper zone on F.Cu, net -BATT
- added copper zone on F.Cu, net Net-(Q101-Pad2)
- removed copper zone on F.Cu, net SHUNT+
- removed copper zone on F.Cu, net SHUNT-
