File: 103_BatteryJunctionBox_BJB/KiCAD/V0_1/BatteryJunctionBox_BJB.sch (KiCad schematic (older format))
At the start: 1 part

Commit message: Mon. Done a Lot of recouvery
Parts:
- removed IC?: LTC2946, _Package_MSOP:MSOP_16_Lead_Plastic, symbol _Measurement_ICs:LTC2946
- added IC101: VOM1271T, _Package_SOP:SOP-4, symbol _Optocoupler:VOM1271T
- added J101, J102, J103, J104: WuertHA_7461057, _Connectors:WuertHA_7461057, symbol _Connector:WuertHA_7461057
- added J105: RJ45_Shielded, Connector_RJ:RJ45_Amphenol_RJHSE5380, symbol Connector:RJ45_Shielded
- added Q101, Q102, Q103, Q104: Q_NMOS_GDS, Package_TO_SOT_SMD:TO-263-3_TabPin2, symbol Device:Q_NMOS_GDS
- added R101: 0.001, _Shunts:R_Shunt_16x8-75_Bourns_4Pin, symbol Device:R_Shunt
- added R102, R103: 10k, Resistor_SMD:R_0805_2012Metric_Pad1.20x1.40mm_HandSolder, symbol Device:R_Small
- added U101: NSL-32, OptoDevice:Luna_NSL-32, symbol Isolator:NSL-32
- added U102: ISO1541, Package_SO:SOIC-8_3.9x4.9mm_P1.27mm, symbol Isolator:ISO1541
Connections:
- new net: J102.1, J102.2, J102.3, J102.4, J102.5, J102.6, Q102.2 (D), Q104.2 (D)
- new net +3V3: J105.7, U101.3 (R), U102.1 (VCC1)
- new net +5V: R102.1, R103.1, U101.1 (A), U102.8 (VCC2)
- new net +BATT: J101.1, J101.2, J101.3, J101.4, J101.5, J101.6, R101.1, R101.2
- new net -BATT: J103.1, J103.2, J103.3, J103.4, J103.5, J103.6, J104.1, J104.2, J104.3, J104.4, J104.5, J104.6, U102.5 (GND2)
- new net I2C_SCL: R103.2, U102.6 (SCL2)
- new net I2C_SCL_ISO: J105.4, U102.3 (SCL1)
- new net I2C_SDA: R102.2, U102.7 (SDA2)
- new net I2C_SDA_ISO: J105.3, U102.2 (SDA1)
- new net ISO_+5V: J105.1
- new net ISO_GND: IC101.2 (K), J105.2, J105.8, U102.4 (GND1)
- new net Interrupt_NO: J105.5, U101.4 (R)
- new net MOSFET_G: IC101.4 (LOAD_2), Q101.1 (G), Q102.1 (G), Q103.1 (G), Q104.1 (G)
- new net MOSFET_S: IC101.3 (LOAD_1), Q101.3 (S), Q102.3 (S), Q103.3 (S), Q104.3 (S)
- new net MOSFET_SWITCH: IC101.1 (A), J105.6
- new net SHUNT-: Q101.2 (D), Q103.2 (D), R101.3, R101.4
- new net ~ALERT: U101.2 (K)
Other:
- note added: "-> To MCU\n"
- note added: "BATTERY\n"
- note added: "LOAD\n"
- note added: "V_ds = 100V\nI_d = 130A\nR_ds(on) = 2mOhm\n \n"

Commit message: some small chages in 7CBS
Connections:
- net +BATT: no longer R101.2
- net SHUNT-: no longer Q101.2 (D), Q103.2 (D), R101.4
- new net: Q101.2 (D), Q103.2 (D), R101.4
- new net SHUNT+: R101.2
Changed lines of the file:
@@
 Wire Wire Line
 	2650 1550 2650 1500
-Wire Wire Line
-	2650 1500 2550 1500
-Wire Wire Line
-	2550 1500 2550 1350
-Connection ~ 2650 1500
-Connection ~ 2550 1350
-Wire Wire Line
-	2850 1500 2950 1500
-Wire Wire Line
-	2950 1500 2950 1350
-Connection ~ 2850 1500
-Connection ~ 2950 1350
 $EndSCHEMATC
